File: hybrid-resistor-mosfet-simulate/hybrid-resistor-mosfet-simulate.kicad_sch (KiCad schematic)
At the start: 0 parts

Commit message: Simple voltage source
Parts:
- added R1: R, symbol Device:R
- added V1: 4.2, symbol Simulation_SPICE:VDC
Connections:
- new net: R1.1, V1.1
- new net GND: R1.2, V1.2

Commit message: Update gitignore
Parts:
- R1: value R -> 1
Other:
- note added: "*.TRAN TSTEP TSTOP <TSTART <TMAX>> <UIC>"
- note added: ".tran 0.1 1 0"
- moved on the sheet: R1
Changed lines of the file:
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@@
 	(generator_version "9.0")
 	(paper "A4")
-	(wire
-		(pts
-			(xy 43.18 58.42) (xy 60.96 58.42)
+	(text ".tran 0.1 1 0"
+		(exclude_from_sim no)
+		(at 107.696 58.928 0)
+		(effects
+			(font
+				(size 1.27 1.27)
+			)
+		)
+	)
+	(text "*.TRAN TSTEP TSTOP <TSTART <TMAX>> <UIC>"
+		(exclude_from_sim no)
+		(at 123.444 64.77 0)
+		(effects
+			(font
+				(size 1.27 1.27)
+			)
+		)
+	)
+	(wire
+		(pts
+			(xy 43.18 58.42) (xy 55.88 58.42)
 		)
 		(stroke
@@
 	(wire
 		(pts
-			(xy 68.58 58.42) (xy 78.74 58.42)
+			(xy 63.5 58.42) (xy 78.74 58.42)
 		)
 		(stroke
@@
 	(symbol
 		(lib_id "Device:R")
-		(at 64.77 58.42 90)
+		(at 59.69 58.42 90)
 		(unit 1)
 		(exclude_from_sim no)
@@
 		(fields_autoplaced yes)
 		(property "Reference" "R1"
-			(at 64.77 52.07 90)
-			(effects
-				(font
-					(size 1.27 1.27)
-				)
-			)
-		)
-		(property "Value" "R"
-			(at 64.77 54.61 90)
+			(at 59.69 52.07 90)
+			(effects
+				(font
+					(size 1.27 1.27)
+				)
+			)
+		)
+		(property "Value" "1"
+			(at 59.69 54.61 90)
 			(effects
 				(font
@@
 		)
 		(property "Footprint" ""
-			(at 64.77 60.198 90)
+			(at 59.69 60.198 90)
 			(effects
 				(font
@@
 		)
 		(property "Datasheet" "~"
-			(at 64.77 58.42 0)
+			(at 59.69 58.42 0)
 			(effects
 				(font
@@
 		)
 		(property "Description" "Resistor"
-			(at 64.77 58.42 0)
-			(effects
-				(font
+			(at 59.69 58.42 0)
+			(effects
+				(font

Commit message: add ignore
Parts:
- removed R1: 1, symbol Device:R
- removed V1: 4.2, symbol Simulation_SPICE:VDC
- added Q1: NMOS, symbol Simulation_SPICE:NMOS
- added R2: 10m, symbol Device:R
- added U1: LM741, symbol Amplifier_Operational:LM741
- added V2: 0.5, symbol Simulation_SPICE:VDC
Connections:
- net GND: now also R2.2, U1.4 (V-), V2.2
- new net: Q1.3 (S), R2.1, U1.2 (-)
- new net: U1.3 (+), V2.1
- new net: Q1.2 (G), U1.6
- new net +5V: U1.7 (V+)
- new net VBUS: Q1.1 (D)
- no-connect marks 0 -> 2
