File: hybrid-resistor-mosfet-simulate/hybrid-resistor-mosfet-simulate.kicad_sch (KiCad schematic)
At the start: 11 parts, among them Q1 NMOS, U2 ${SIM.PARAMS}

Commit message: Tuning the LC value
Parts:
- added C3: 470u, symbol Device:C
- added L1: 500n, symbol Device:L
Connections:
- net GND: now also C3.2
- net VBUS: now also L1.1; no longer Q1.1 (D)
- new net: C3.1, L1.2, Q1.1 (D)
Other:
- note added: ".tran 10n 10m 0"
- note removed: ".tran 0.1 1 0"
