File: hybrid-resistor-mosfet-simulate/hybrid-resistor-mosfet-simulate.kicad_sch (KiCad schematic)
At the start: 13 parts, among them Q1 NMOS, U2 ${SIM.PARAMS}

Commit message: create load board v1
Parts:
- added R5: 100m, symbol Device:R
- C2: value 100n -> 50n
- L1: value 500n -> 50n
Connections:
- net VBUS: now also R5.1; no longer V3.1
- new net: R5.2, V3.1
Changed lines of the file:
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@@
+	)
+	(junction
+		(at 100.33 116.84)
+		(diameter 0)
+		(color 0 0 0 0)
+	)
+	(junction
+		(at 100.33 133.35)
+		(diameter 0)
+		(color 0 0 0 0)
 	)
 	(junction
@@
 	)
 	(junction
-		(at 101.6 133.35)
-		(diameter 0)
-		(color 0 0 0 0)
-	)
-	(junction
-		(at 101.6 116.84)
-		(diameter 0)
-		(color 0 0 0 0)
-	)
-	(junction
 		(at 90.17 101.6)
 		(diameter 0)
@@
 	(wire
 		(pts
-			(xy 101.6 116.84) (xy 109.22 116.84)
+			(xy 85.09 133.35) (xy 85.09 119.38)
 		)
 		(stroke
@@
 	(wire
 		(pts
-			(xy 85.09 133.35) (xy 85.09 119.38)
+			(xy 128.27 133.35) (xy 128.27 137.16)
 		)
 		(stroke
@@
 	(wire
 		(pts
-			(xy 128.27 133.35) (xy 128.27 137.16)
+			(xy 119.38 116.84) (xy 120.65 116.84)
 		)
 		(stroke
@@
 	(wire
 		(pts
-			(xy 119.38 116.84) (xy 120.65 116.84)
+			(xy 90.17 101.6) (xy 101.6 101.6)
 		)
 		(stroke
@@
 	(wire
 		(pts
-			(xy 90.17 101.6) (xy 101.6 101.6)
+			(xy 128.27 121.92) (xy 128.27 133.35)
 		)
 		(stroke
@@
 	(wire
 		(pts
-			(xy 128.27 121.92) (xy 128.27 133.35)
+			(xy 100.33 116.84) (xy 109.22 116.84)
 		)
 		(stroke
@@
 	(wire
 		(pts
-			(xy 100.33 116.84) (xy 101.6 116.84)
+			(xy 100.33 116.84) (xy 100.33 120.65)
 		)
 		(stroke
@@
 	(wire
 		(pts
-			(xy 85.09 133.35) (xy 101.6 133.35)
+			(xy 158.75 114.3) (xy 158.75 115.57)
 		)
 		(stroke
@@
 	(wire
 		(pts
-			(xy 101.6 133.35) (xy 106.68 133.35)
+			(xy 158.75 105.41) (xy 158.75 106.68)
 		)
 		(stroke
@@
 	(wire
 		(pts
-			(xy 101.6 124.46) (xy 101.6 133.35)
+			(xy 100.33 133.35) (xy 106.68 133.35)
 		)
 		(stroke
@@
 	(wire
 		(pts
-			(xy 158.75 105.41) (xy 158.75 115.57)
+			(xy 100.33 128.27) (xy 100.33 133.35)
 		)
 		(stroke
@@
 	(wire
 		(pts
-			(xy 128.27 111.76) (xy 144.78 111.76)
+			(xy 85.09 133.35) (xy 100.33 133.35)
 		)
 		(stroke
@@
 		)
 	)
+	(wire
+		(pts
+			(xy 128.27 111.76) (xy 144.78 111.76)
+		)
+		(stroke
+			(width 0)
+			(type default)
+		)
+	)
+	(symbol
+		(lib_id "Device:R")
+		(at 158.75 110.49 0)
+		(unit 1)
+		(exclude_from_sim no)
+		(in_bom yes)
+		(on_board yes)
+		(dnp no)
+		(fields_autoplaced yes)
+		(property "Reference" "R5"
+			(at 161.29 109.2199 0)
+			(effects
+				(font
+					(size 1.27 1.27)
+				)
+				(justify left)
+			)
+		)
+		(property "Value" "100m"
+			(at 161.29 111.7599 0)
+			(effects
+				(font
+					(size 1.27 1.27)
+				)
+				(justify left)
+			)
+		)
+		(property "Footprint" ""
+			(at 156.972 110.49 90)
+			(effects
+				(font
+					(size 1.27 1.27)
+				)
+				(hide yes)
+			)
+		)
+		(property "Datasheet" "~"
+			(at 158.75 110.49 0)
+			(effects
+				(font
+					(size 1.27 1.27)
+				)
+				(hide yes)
+			)
+		)
+		(property "Description" "Resistor"
+			(at 158.75 110.49 0)
+			(effects
+				(font
+					(size 1.27 1.27)
+				)
+				(hide yes)
+			)
+		)
+		(pin "2"
+		)
+		(pin "1"
+		)
+		(instances
+			(project ""
+				(path "/f84774a7-5641-4a3c-9dbb-5b6461eb80bc"
+					(reference "R5")
+					(unit 1)
+				)
+			)
+		)
+	)
 	(symbol
 		(lib_id "power:GND")
@@
 	)
 	(symbol
-		(lib_id "Device:C")
-		(at 101.6 120.65 0)
-		(unit 1)
-		(exclude_from_sim no)
-		(in_bom yes)
-		(on_board yes)
-		(dnp no)
-		(fields_autoplaced yes)
-		(property "Reference" "C2"
-			(at 105.41 119.3799 0)
-			(effects
-				(font
-					(size 1.27 1.27)
-				)
-				(justify left)
-			)
-		)
-		(property "Value" "100n"
-			(at 105.41 121.9199 0)
-			(effects
-				(font
-					(size 1.27 1.27)
-				)
-				(justify left)
-			)
-		)
-		(property "Footprint" ""
-			(at 102.5652 124.46 0)
-			(effects
-				(font
-					(size 1.27 1.27)
-				)
-				(hide yes)
-			)
-		)
-		(property "Datasheet" "~"
-			(at 101.6 120.65 0)
-			(effects
-				(font
-					(size 1.27 1.27)
-				)
-				(hide yes)
-			)
-		)
-		(property "Description" "Unpolarized capacitor"
-			(at 101.6 120.65 0)
-			(effects
-				(font
-					(size 1.27 1.27)
-				)
-				(hide yes)
-			)
-		)
-		(property "Sim.Device" "C"
-			(at 0 0 0)
-			(effects
-				(font
-					(size 1.27 1.27)
-				)
-				(hide yes)
-			)
-		)
-		(property "Sim.Pins" "1=+ 2=-"
-			(at 0 0 0)
-			(effects
-				(font
-					(size 1.27 1.27)
-				)
-				(hide yes)
-			)
-		)
-		(pin "2"
-		)
-		(pin "1"
-		)
-		(instances
-			(project ""
-				(path "/f84774a7-5641-4a3c-9dbb-5b6461eb80bc"
-					(reference "C2")
-					(unit 1)
-				)
-			)
-		)
-	)
-	(symbol
 		(lib_id "power:GND")
 		(at 144.78 119.38 0)
@@
 		(on_board yes)
 		(dnp no)
-		(fields_autoplaced yes)
 		(property "Reference" "R1"
-			(at 110.49 127 90)
+			(at 110.49 129.286 90)
 			(effects
 				(font
@@
 		)
 		(property "Value" "500"
-			(at 110.49 129.54 90)
+			(at 109.728 131.064 90)
 			(effects
 				(font
@@
 			)
 		)
-		(property "Value" "500n"
+		(property "Value" "50n"
 			(at 129.54 109.2199 0)
 			(effects
@@
 					(unit 1)
 				)
+			)
+		)
+	)
+	(symbol
+		(lib_id "Device:C")
+		(at 100.33 124.46 0)
+		(unit 1)
+		(exclude_from_sim no)
+		(in_bom yes)
+		(on_board yes)
+		(dnp no)
+		(property "Reference" "C2"
+			(at 101.346 122.428 0)
+			(effects
+				(font
+					(size 1.27 1.27)
+				)
+				(justify left)
+			)
+		)
+		(property "Value" "50n"
+			(at 101.6 126.492 0)
+			(effects
+				(font
+					(size 1.27 1.27)
+				)
+				(justify left)
+			)
+		)
+		(property "Footprint" ""
+			(at 101.2952 128.27 0)
+			(effects
+				(font
+					(size 1.27 1.27)
+				)
+				(hide yes)
+			)
+		)
+		(property "Datasheet" "~"
+			(at 100.33 124.46 0)
+			(effects
+				(font
+					(size 1.27 1.27)
+				)
+				(hide yes)
+			)
+		)
+		(property "Description" "Unpolarized capacitor"
+			(at 100.33 124.46 0)
+			(effects
+				(font
+					(size 1.27 1.27)
+				)
+				(hide yes)
+			)
+		)
+		(pin "1"
+		)
+		(pin "2"
+		)
+		(instances
+			(project ""
+				(path "/f84774a7-5641-4a3c-9dbb-5b6461eb80bc"
+					(reference "C2")
+					(unit 1)
+				)
